File: hardware/flowerinator/flowerinator.kicad_sch (KiCad schematic)
At the start: 0 parts

Commit message: some tidying up
Parts:
- added 1: Water Pump, symbol lib:Water_Pump
- added U1: ESP32-WROOM-32, RF_Module:ESP32-WROOM-32, symbol RF_Module:ESP32-WROOM-32
Connections:
- new net GND: U1.1 (GND), U1.15 (GND), U1.38 (GND), U1.39 (GND)
