File: hardware/flowerinator.kicad_pcb (KiCad board)
At the start: 2 copper layers, 13 parts, among them J10 Screw_Terminal_01x03, J2 Screw_Terminal_01x02, J3 Screw_Terminal_01x02, J4 Screw_Terminal_01x02, J5 Screw_Terminal_01x03, J6 Screw_Terminal_01x03, J7 Screw_Terminal_01x03, J8 Screw_Terminal_01x03, J9 Screw_Terminal_01x05, Q2 FDMS8350LET40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

Commit message: exported the pcb
Parts:
- moved J10 72.2 mm to (139.6, 143.0)
- moved J2 72.2 mm to (176.9, 100.0)
- moved J3 72.2 mm to (176.9, 86.8)
- moved J4 72.2 mm to (177.0, 74.1)
- moved J5 72.2 mm to (130.4, 129.0)
- moved J6 72.2 mm to (141.5, 129.0)
- moved J7 72.2 mm to (152.6, 129.0)
- moved J8 72.2 mm to (163.6, 129.0)
- moved J9 72.2 mm to (176.6, 144.0)
- moved Q2 72.2 mm to (155.6, 100.5)
- moved Q3 72.2 mm to (155.6, 87.0)
- moved Q4 72.2 mm to (155.6, 74.0)
- moved U6 72.2 mm to (121.8, 67.3)
Routing:
- net Net-(J2-Pin_2): track 15.1 -> 22.1 mm
- net Net-(J3-Pin_2): track 15.0 -> 19.9 mm
- net Net-(J4-Pin_2): track 15.0 -> 19.9 mm
- net Net-(Q3-G): track 28.6 -> 27.9 mm
- net Net-(Q2-G): track 18.5 -> 17.7 mm
- net Net-(Q4-G): track 28.9 -> 28.2 mm
Other:
- board text added: "Grow lights"
- board text added: "Motor"
- board text added: "Pump"
- board text added: "Soil sensor 1"
- board text added: "Soil sensor 2"
- board text added: "Touch sensor"
- board text added: "Ultrasonic sensor"
- board text added: "Water sensor"
